File: Schematic & PCB (current)/zynqPCB-master/power.kicad_sch (KiCad schematic)
At the start: 58 parts, among them CON1 AVR-JTAG-10, U1 LM3880, U2 LM3880, U20 xc7z020clg484, U3 SC189 - 1.0V, U4 SC189 - 3.3V, U5 TLV62080DSGx, U7 SC189 - 1.8V

Commit message: 8/1 update
Parts:
- removed R88, R89, R90: .05, Resistor_SMD:R_2512_6332Metric, symbol DFTCustom:R
Connections:
- net 1V35_CS is gone; now on net +5V: C108.1, U5.8 (VIN)
- net 1V8_CS is gone; now on net +5V: C13.1, U7.1 (VIN)
- net 3V3_CS is gone; now on net +5V: C3.1, U4.1 (VIN)
Changed lines of the file:
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@@
     )
   )
-  (symbol (lib_id "power:+5V") (at 99.06 66.04 0) (unit 1)
-    (in_bom yes) (on_board yes) (dnp no)
-    (property "Reference" "#PWR028" (at 99.06 63.754 0)
+  (symbol (lib_id "power:+5V") (at 99.06 73.66 0) (unit 1)
+    (in_bom yes) (on_board yes) (dnp no)
+    (property "Reference" "#PWR028" (at 99.06 71.374 0)
       (effects (font (size 0.508 0.508)) hide)
     )
-    (property "Value" "+5V" (at 99.06 63.754 0)
+    (property "Value" "+5V" (at 99.06 71.374 0)
       (effects (font (size 0.762 0.762)))
     )
-    (property "Footprint" "" (at 99.06 66.04 0)
-      (effects (font (size 1.524 1.524)) hide)
-    )
-    (property "Datasheet" "" (at 99.06 66.04 0)
+    (property "Footprint" "" (at 99.06 73.66 0)
+      (effects (font (size 1.524 1.524)) hide)
+    )
+    (property "Datasheet" "" (at 99.06 73.66 0)
       (effects (font (size 1.524 1.524)) hide)
     )
@@
     )
   )
-  (symbol (lib_id "DFTCustom:R") (at 99.06 69.85 0) (unit 1)
-    (in_bom yes) (on_board yes) (dnp no)
-    (property "Reference" "R90" (at 100.838 68.6816 0)
-      (effects (font (size 1.27 1.27)) (justify left))
-    )
-    (property "Value" ".05" (at 100.838 70.993 0)
-      (effects (font (size 1.27 1.27)) (justify left))
-    )
-    (property "Footprint" "Resistor_SMD:R_2512_6332Metric" (at 97.282 69.85 90)
-      (effects (font (size 1.27 1.27)) hide)
-    )
-    (property "Datasheet" "" (at 99.06 69.85 0)
-      (effects (font (size 1.27 1.27)) hide)
-    )
-    (property "MFR" "Bourns Inc" (at 0 139.7 0)
-      (effects (font (size 1.27 1.27)) hide)
-    )
-    (property "MPN" "CRA2512-FZ-R050ELF" (at 0 139.7 0)
-      (effects (font (size 1.27 1.27)) hide)
-    )
-    (property "SPR" "Digikey" (at 0 139.7 0)
-      (effects (font (size 1.27 1.27)) hide)
-    )
-    (property "SPN" "CRA2512-FZ-R050ELFCT-ND" (at 0 139.7 0)
-      (effects (font (size 1.27 1.27)) hide)
-    )
-    (property "SPURL" "-" (at 0 139.7 0)
-      (effects (font (size 1.27 1.27)) hide)
-    )
-    (pin "1")
-    (pin "2")
-    (instances
-      (project "DFTBoard"
-        (path "/b8a438e2-fdd4-4382-b8df-6f293dcfe534/00000000-0000-0000-0000-000058508414"
-          (reference "R90") (unit 1)
-        )
-      )
-    )
-  )
-  (symbol (lib_id "power:+5V") (at 15.24 36.83 0) (unit 1)
-    (in_bom yes) (on_board yes) (dnp no)
-    (property "Reference" "#PWR04" (at 15.24 34.544 0)
+  (symbol (lib_id "power:+5V") (at 15.24 44.45 0) (unit 1)
+    (in_bom yes) (on_board yes) (dnp no)
+    (property "Reference" "#PWR04" (at 15.24 42.164 0)
       (effects (font (size 0.508 0.508)) hide)
     )
-    (property "Value" "+5V" (at 15.24 34.544 0)
+    (property "Value" "+5V" (at 15.24 42.164 0)
       (effects (font (size 0.762 0.762)))
     )
-    (property "Footprint" "" (at 15.24 36.83 0)
-      (effects (font (size 1.524 1.524)) hide)
-    )
-    (property "Datasheet" "" (at 15.24 36.83 0)
+    (property "Footprint" "" (at 15.24 44.45 0)
+      (effects (font (size 1.524 1.524)) hide)
+    )
+    (property "Datasheet" "" (at 15.24 44.45 0)
       (effects (font (size 1.524 1.524)) hide)
     )
@@
         (path "/b8a438e2-fdd4-4382-b8df-6f293dcfe534/00000000-0000-0000-0000-000058508414"
           (reference "#PWR04") (unit 1)
-        )
-      )
-    )
-  )
-  (symbol (lib_id "DFTCustom:R") (at 15.24 40.64 0) (unit 1)
-    (in_bom yes) (on_board yes) (dnp no)
-    (property "Reference" "R88" (at 17.018 39.4716 0)
-      (effects (font (size 1.27 1.27)) (justify left))
-    )
-    (property "Value" ".05" (at 17.018 41.783 0)
-      (effects (font (size 1.27 1.27)) (justify left))
-    )
-    (property "Footprint" "Resistor_SMD:R_2512_6332Metric" (at 13.462 40.64 90)
-      (effects (font (size 1.27 1.27)) hide)
-    )
-    (property "Datasheet" "" (at 15.24 40.64 0)
-      (effects (font (size 1.27 1.27)) hide)
-    )
-    (property "MFR" "Bourns Inc" (at 0 81.28 0)
-      (effects (font (size 1.27 1.27)) hide)
-    )
-    (property "MPN" "CRA2512-FZ-R050ELF" (at 0 81.28 0)
-      (effects (font (size 1.27 1.27)) hide)
-    )
-    (property "SPR" "Digikey" (at 0 81.28 0)
-      (effects (font (size 1.27 1.27)) hide)
-    )
-    (property "SPN" "CRA2512-FZ-R050ELFCT-ND" (at 0 81.28 0)
-      (effects (font (size 1.27 1.27)) hide)
-    )
-    (property "SPURL" "-" (at 0 81.28 0)
-      (effects (font (size 1.27 1.27)) hide)
-    )
-    (pin "1")
-    (pin "2")
-    (instances
-      (project "DFTBoard"
-        (path "/b8a438e2-fdd4-4382-b8df-6f293dcfe534/00000000-0000-0000-0000-000058508414"
-          (reference "R88") (unit 1)
         )
       )
@@
     )
   )
-  (symbol (lib_id "power:+5V") (at 29.21 110.49 90) (unit 1)
-    (in_bom yes) (on_board yes) (dnp no)
-    (property "Reference" "#PWR010" (at 26.924 110.49 0)
+  (symbol (lib_id "power:+5V") (at 36.83 110.49 90) (unit 1)
+    (in_bom yes) (on_board yes) (dnp no)
+    (property "Reference" "#PWR010" (at 34.544 110.49 0)
       (effects (font (size 0.508 0.508)) hide)
     )
-    (property "Value" "+5V" (at 26.924 110.49 0)
+    (property "Value" "+5V" (at 34.544 110.49 0)
       (effects (font (size 0.762 0.762)))
     )
-    (property "Footprint" "" (at 29.21 110.49 0)
-      (effects (font (size 1.524 1.524)) hide)
-    )
-    (property "Datasheet" "" (at 29.21 110.49 0)
+    (property "Footprint" "" (at 36.83 110.49 0)
+      (effects (font (size 1.524 1.524)) hide)
+    )
+    (property "Datasheet" "" (at 36.83 110.49 0)
       (effects (font (size 1.524 1.524)) hide)
     )
@@
         )
       )
-    )
-  )
-  (symbol (lib_id "DFTCustom:R") (at 33.02 110.49 90) (unit 1)
-    (in_bom yes) (on_board yes) (dnp no)
-    (property "Reference" "R89" (at 31.8516 108.712 0)
-      (effects (font (size 1.27 1.27)) (justify left))
-    )
-    (property "Value" ".05" (at 34.163 108.712 0)
-      (effects (font (size 1.27 1.27)) (justify left))
-    )
-    (property "Footprint" "Resistor_SMD:R_2512_6332Metric" (at 33.02 112.268 90)
-      (effects (font (size 1.27 1.27)) hide)
-    )
-    (property "Datasheet" "" (at 33.02 110.49 0)
-      (effects (font (size 1.27 1.27)) hide)
-    )
-    (property "MFR" "Bourns Inc" (at 143.51 143.51 0)
-      (effects (font (size 1.27 1.27)) hide)
-    )
-    (property "MPN" "CRA2512-FZ-R050ELF" (at 143.51 143.51 0)
-      (effects (font (size 1.27 1.27)) hide)
-    )
-    (property "SPR" "Digikey" (at 143.51 143.51 0)
-      (effects (font (size 1.27 1.27)) hide)
-    )
-    (property "SPN" "CRA2512-FZ-R050ELFCT-ND" (at 143.51 143.51 0)
-      (effects (font (size 1.27 1.27)) hide)
-    )
-    (property "SPURL" "-" (at 143.51 143.51 0)
-      (effects (font (size 1.27 1.27)) hide)
-    )
-    (pin "1")
-    (pin "2")
-    (instances
-      (project "DFTBoard"
-        (path "/b8a438e2-fdd4-4382-b8df-6f293dcfe534/00000000-0000-0000-0000-000058508414"
-          (reference "R89") (unit 1)
-        )
-      )
