File: Prototype Breadboard/FPGApwr.kicad_sch (KiCad schematic)
At the start: 21 parts, among them J6 Conn_01x04_MountingPin, U3 XC7Z010-1CLG225I

Commit message: 1/4 update
update the breadboard version
Parts:
- removed C23: 4.7uF, Capacitor_SMD:C_0402_1005Metric, symbol Device:C
- J6: footprint Connector_PinSocket_2.54mm:PinSocket_2x02_P2.54mm_Vertical -> Connector_PinSocket_2.54mm:PinSocket_1x04_P2.54mm_Vertical
Connections:
- net GPIO12: now also J6.2 (Pin_2), U3.L9 (TMS_0); no longer J6.4 (Pin_4), U3.L7 (TDI_0)
- net GPIO14: now also J6.4 (Pin_4), U3.L7 (TDI_0); no longer J6.2 (Pin_2), U3.L9 (TMS_0)
Changed lines of the file:
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@@
 	)
 	(junction
-		(at 257.81 27.94)
-		(diameter 0)
-		(color 0 0 0 0)
-	)
-	(junction
 		(at 201.93 30.48)
 		(diameter 0)
@@
 	(wire
 		(pts
-			(xy 257.81 27.94) (xy 261.62 27.94)
+			(xy 250.19 27.94) (xy 261.62 27.94)
 		)
 		(stroke
@@
 	(wire
 		(pts
-			(xy 250.19 27.94) (xy 257.81 27.94)
-		)
-		(stroke
-			(width 0)
-			(type default)
-		)
-	)
-	(wire
-		(pts
 			(xy 173.99 88.9) (xy 177.8 88.9)
 		)
@@
 		)
 	)
-	(global_label "GPIO12"
+	(global_label "GPIO14"
 		(shape bidirectional)
 		(at 35.052 43.18 180)
@@
 		)
 	)
-	(global_label "GPIO14"
+	(global_label "GPIO12"
 		(shape bidirectional)
 		(at 35.052 40.64 180)
@@
 			)
 		)
-		(property "Footprint" "Connector_PinSocket_2.54mm:PinSocket_2x02_P2.54mm_Vertical"
+		(property "Footprint" "Connector_PinSocket_2.54mm:PinSocket_1x04_P2.54mm_Vertical"
 			(at 41.91 29.21 0)
 			(effects
@@
 					(unit 1)
 				)
-			)
-		)
-	)
-	(symbol
-		(lib_id "Device:C")
-		(at 257.81 31.75 0)
-		(unit 1)
-		(exclude_from_sim no)
-		(in_bom yes)
-		(on_board yes)
-		(dnp no)
-		(property "Reference" "C23"
-			(at 261.62 30.4799 0)
-			(effects
-				(font
-					(size 1.27 1.27)
-				)
-				(justify left)
-				(hide yes)
-			)
-		)
-		(property "Value" "4.7uF"
-			(at 258.572 34.29 0)
-			(effects
-				(font
-					(size 1.27 1.27)
-				)
-				(justify left)
-			)
-		)
-		(property "Footprint" "Capacitor_SMD:C_0402_1005Metric"
-			(at 258.7752 35.56 0)
-			(effects
-				(font
-					(size 1.27 1.27)
-				)
-				(hide yes)
-			)
-		)
-		(property "Datasheet" "~"
-			(at 257.81 31.75 0)
-			(effects
-				(font
-					(size 1.27 1.27)
-				)
-				(hide yes)
-			)
-		)
-		(property "Description" "Unpolarized capacitor"
-			(at 257.81 31.75 0)
-			(effects
-				(font
-					(size 1.27 1.27)
-				)
-				(hide yes)
-			)
-		)
-		(property "LCSC" ""
-			(at 257.81 31.75 0)
-			(effects
-				(font
-					(size 1.27 1.27)
-				)
-				(hide yes)
-			)
-		)
-		(pin "2"
-		)
-		(pin "1"
-		)
-		(instances
-			(project "SYNC-VT"
-				(path "/8b98976c-b0e2-4979-aa9a-b6389ce6c189/e0fdbcfa-176a-4d8c-897b-d3b34c4c4b6c"
-					(reference "C23")
-					(unit 1)
-				)
