File: Prototype Breadboard/Power.kicad_sch (KiCad schematic)
At the start: 39 parts, among them U1 MPM3834CGPA-Z, U11 SC189ZULTRT-3v3, U2 MPM3834CGPA-Z, U4 TPS3106K33DBVR, U8 ZL6201A33S3

Commit message: 1/4 update
update the breadboard version
Parts:
- D4: footprint Diode_SMD:D_SOD-523 -> Diode_SMD:D_SMA
Connections:
- net +3V3: no longer C10.1, C8.1, R4.2, R6.2, U1.12 (IN), U1.13 (IN), U1.14 (IN), U1.3 (EN), U2.12 (IN), U2.13 (IN), U2.14 (IN), U2.3 (EN)
- net +5VD: now reaches C36.2, D4.1 (K), U8.3 (VI)
- net +5VD: now also C10.1, C8.1, R4.2, R6.2, U1.12 (IN), U1.13 (IN), U1.14 (IN), U1.3 (EN), U2.12 (IN), U2.13 (IN), U2.14 (IN), U2.3 (EN)
