File: Prototype Breadboard/SYNC-VT.kicad_pcb (KiCad board)
At the start: 6 copper layers, 74.3 x 21 mm, 113 parts, among them J1 Button, J2 Button, J3 Conn_02x06_Odd_Even_MountingP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, J4 Conn_01x23_MountingPin, J5 Conn_01x23_MountingPin, J6 Conn_01x04_MountingPin, U1 MPM3834CGPA-Z, U11 SC189ZULTRT-3v3, U2 MPM3834CGPA-Z, U3 XC7Z010-1CLG225I, U4 TPS3106K33DBVR, U5 W25Q128JVS, U6 0473092651, U7 S80KS5123GABHA020, U8 ZL6201A33S3, U9 RP2040, X1 SIT8008BI-73-XXS-33.333333, Y1 3225-4P 12MHz

Commit message: 1/4 update
update the breadboard version
Parts:
- removed C23: 4.7uF, Capacitor_SMD:C_0402_1005Metric
- added J7: Conn_01x30_MountingPin, Connector_PinHeader_2.54mm:PinHeader_1x30_P2.54mm_Vertical, F.Cu at (152.8, 40.4)
- added J8: Conn_01x24_MountingPin, Connector_FFC-FPC:TE_2-1734839-4_1x24-1MP_P0.5mm_Horizontal, B.Cu at (74.7, 50.4)
- added U10: NanoS3, Sync_VT extras:NanoS3, F.Cu at (89.5, 44.1)
- D4: footprint Diode_SMD:D_SOD-523 -> Diode_SMD:D_SMA
- J3: value Conn_02x06_Odd_Even_MountingPin -> Conn_01x30_MountingPin; footprint Connector_PinSocket_2.54mm:PinSocket_2x06_P2.54mm_Vertical -> Connector_PinHeader_2.54mm:PinHeader_1x30_P2.54mm_Vertical
- J4, J5: value Conn_01x23_MountingPin -> Conn_01x25_MountingPin; footprint Connector_PinHeader_2.54mm:PinHeader_1x23_P2.54mm_Vertical -> Connector_PinHeader_2.54mm:PinHeader_1x25_P2.54mm_Vertical
- J6: footprint Connector_PinSocket_2.54mm:PinSocket_2x02_P2.54mm_Vertical -> Connector_PinSocket_2.54mm:PinSocket_1x04_P2.54mm_Vertical
- R23: moved to F.Cu
- TP1, TP2, TP3, TP4, TP5, TP6, TP7, U5, U7: moved to B.Cu
- moved D4 101.8 mm to (150.7, 54.7)
- moved TP3 77.2 mm to (122.2, 53.2), turned to 180 degrees
- moved J3 74.7 mm to (152.8, 39.0), turned to -90 degrees
- moved TP1 72.1 mm to (114.8, 55.7), turned to 180 degrees
- moved TP2 70.1 mm to (115.3, 48.6), turned to 180 degrees
- moved TP4 69.7 mm to (115.0, 53.7), turned to 180 degrees
- moved TP5 69.1 mm to (115.3, 46.5), turned to 180 degrees
- moved U7 42.8 mm to (87.6, 45.3), turned to -90 degrees
- moved U5 37.3 mm to (87.1, 51.7)
- moved TP6 31.1 mm to (151.1, 45.8), turned to 180 degrees
- moved TP7 31.0 mm to (151.1, 48.7), turned to 180 degrees
- moved TP11 31.0 mm to (122.9, 55.3), turned to 180 degrees
- moved TP10 30.6 mm to (125.5, 55.3), turned to 180 degrees
- moved J6 19.5 mm to (78.7, 58.7), turned to 90 degrees
- moved R23 18.8 mm to (106.2, 56.1)
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Connections:
- C10 pad 1: +3V3 -> +5VD
- C36 pad 2: Net-(D4-K) -> +5VD
- C8 pad 1: +3V3 -> +5VD
- D4 pad 1: Net-(D4-K) -> +5VD
- J3 pad 1: +3V3 -> VBUS0
- J3 pad 10: IO1P -> GPIO6
- J3 pad 11: IOL5N -> GPIO7
- J3 pad 12: IO3P -> IO21P
- J3 pad 2: +3V3 -> GND
- J3 pad 3: GND -> +3.3VA
- J3 pad 4: GND -> GPIO0
- J3 pad 5: IO5N -> GPIO1
- J3 pad 6: IO5P -> GPIO2
- J3 pad 7: IO3N -> GPIO3
- J3 pad 8: IO2P -> GPIO4
- J3 pad 9: IOL5P -> GPIO5
- J4 pad 10: GPIO6 -> GPIO23
- J4 pad 11: GPIO7 -> GPIO22
- J4 pad 12: IO8N -> MIO13
- J4 pad 13: IO9N -> MIO9
- J4 pad 14: IO7N -> MIO10
- J4 pad 15: IO15P -> GND
- J4 pad 16: IO15N -> MIO48
- J4 pad 17: IO7P -> MIO52
- J4 pad 18: IO18N -> MIO14
- J4 pad 19: IO17N -> MIO11
- J4 pad 20: IO18P -> GND
- J4 pad 21: IO17P -> MIO36
- J4 pad 22: IO13N -> MIO35
- J4 pad 23: IO16N -> MIO53
- J4 pad 4: GPIO0 -> GPIO29
- J4 pad 5: GPIO1 -> GPIO28
- J4 pad 6: GPIO2 -> GPIO27
- J4 pad 7: GPIO3 -> GPIO26
- J4 pad 8: GPIO4 -> GPIO25
- J4 pad 9: GPIO5 -> GPIO24
- J5 pad 12: MIO34 -> MIO13
- J5 pad 13: MIO35 -> MIO9
- J5 pad 14: MIO36 -> MIO10
- J5 pad 15: MIO37 -> GND
- J5 pad 16: MIO39 -> MIO48
- J5 pad 17: MIO38 -> MIO52
- J5 pad 18: MIO41 -> MIO14
- J5 pad 19: MIO43 -> MIO11
- J5 pad 20: MIO42 -> GND
- J5 pad 21: MIO40 -> MIO36
- J5 pad 22: MIO11 -> MIO35
- J5 pad 23: MIO14 -> MIO53
- J6 pad 2: GPIO14 -> GPIO12
- J6 pad 4: GPIO12 -> GPIO14
- R4 pad 2: +3V3 -> +5VD
- R6 pad 2: +3V3 -> +5VD
- U1 pad 12: +3V3 -> +5VD
- U1 pad 13: +3V3 -> +5VD
- U1 pad 14: +3V3 -> +5VD
- U1 pad 3: +3V3 -> +5VD
- U2 pad 12: +3V3 -> +5VD
- U2 pad 13: +3V3 -> +5VD
- U2 pad 14: +3V3 -> +5VD
- U2 pad 3: +3V3 -> +5VD
- U3 pad A12: MIO42 -> MIO52
- U3 pad A13: MIO38 -> unconnected-(U3D-PS_MIO38_501-PadA13)
- U3 pad A14: MIO39 -> MIO35
- U3 pad B12: MIO40 -> MIO48
- U3 pad B14: MIO37 -> MIO36
- U3 pad B5: unconnected-(U3D-PS_MIO9_500-PadB5) -> MIO9
- U3 pad C13: MIO43 -> MIO53
- U3 pad C14: MIO36 -> MIO37
- U3 pad C6: unconnected-(U3D-PS_MIO13_500-PadC6) -> MIO13
- U3 pad D13: MIO41 -> unconnected-(U3D-PS_MIO49_501-PadD13)
- U3 pad D14: MIO35 -> MIO39
- U3 pad D6: unconnected-(U3D-PS_MIO10_500-PadD6) -> MIO10
- U3 pad E11: IO2P -> unconnected-(U3C-IO_L2P_T0_AD8P_35-PadE11)
- U3 pad E12: unconnected-(U3C-IO_L2N_T0_AD8N_35-PadE12) -> AIO8N
- U3 pad E13: unconnected-(U3C-IO_L1N_T0_AD0N_35-PadE13) -> AIO0N
- U3 pad F12: IO1P -> unconnected-(U3C-IO_L1P_T0_AD0P_35-PadF12)
- U3 pad F13: IO3P -> AIO3P
- U3 pad F14: IO3N -> AIO3N
- U3 pad F15: IOL5N -> AIO5N
- U3 pad G14: unconnected-(U3B-IO_L3P_T0_DQS_PUDC_B_34-PadG14) -> IO3P
- U3 pad G15: IOL5P -> AIO5P
- U3 pad H11: unconnected-(U3B-IO_L6P_T0_34-PadH11) -> GPIO17
- U3 pad H12: unconnected-(U3B-IO_L1N_T0_34-PadH12) -> IO1N
- U3 pad H13: unconnected-(U3B-IO_L2N_T0_34-PadH13) -> IO2N
- U3 pad H14: unconnected-(U3B-IO_L3N_T0_DQS_34-PadH14) -> IO3N
- U3 pad J15: GPIO17 -> IO4P
- U3 pad K11: unconnected-(U3B-IO_L11P_T1_SRCC_34-PadK11) -> IO11P
- U3 pad K12: unconnected-(U3B-IO_L11N_T1_SRCC_34-PadK12) -> IO11N
- U3 pad K13: unconnected-(U3B-IO_L10P_T1_34-PadK13) -> IO10P
- U3 pad K15: GPIO16 -> IO4N
- U3 pad L12: unconnected-(U3B-IO_L12P_T1_MRCC_34-PadL12) -> IO12P
- U3 pad L13: unconnected-(U3B-IO_L10N_T1_34-PadL13) -> RAM_DQ4
- U3 pad L14: unconnected-(U3B-IO_L9P_T1_DQS_34-PadL14) -> ~{RAM_RST}
- U3 pad L15: unconnected-(U3B-IO_L8P_T1_34-PadL15) -> RWDS
- U3 pad L7: GPIO12 -> GPIO14
- U3 pad L9: GPIO14 -> GPIO12
- U3 pad M10: RAM_DQ2 -> IO21P
- U3 pad M11: RAM_DQ4 -> IO21N
- U3 pad M12: unconnected-(U3B-IO_L12N_T1_MRCC_34-PadM12) -> IO12N
- U3 pad M14: IO9N -> RAM_DQ2
- U3 pad M15: IO8N -> ~{RAM_CS0}
- U3 pad M9: RAM_DQ3 -> GPIO16
- U3 pad N11: ~{RAM_CLK} -> IO13P
- U3 pad N12: IO13N -> RAM_DQ5
- U3 pad N13: IO7P -> RAM_DQ3
- U3 pad N14: IO7N -> RAM_CLK
- U3 pad N7: unconnected-(U3B-IO_L22P_T3_34-PadN7) -> IO22P
- U3 pad N8: RAM_DQ0 -> IO22N
- U3 pad N9: RWDS -> IO19N
- U3 pad P10: RAM_CLK -> IO24P
- U3 pad P11: ~{RAM_RST} -> RAM_DQ6
- U3 pad P13: IO18P -> RAM_DQ0
- U3 pad P15: IO15P -> ~{RAM_CLK}
- U3 pad P8: RAM_DQ6 -> IO23P
- U3 pad P9: RAM_DQ1 -> IO23N
- U3 pad R10: ~{RAM_CS0} -> IO24N
- U3 pad R12: IO17P -> RAM_DQ7
- U3 pad R13: IO17N -> RAM_DQ1
- U3 pad R7: RAM_DQ7 -> IO20P
- U3 pad R8: RAM_DQ5 -> IO20N
- U8 pad 3: Net-(D4-K) -> +5VD
Routing:
- net GPIO15: track 0.00 -> 63.2 mm, vias 0 -> 3
- net GPIO12: track 0.00 -> 59.5 mm, vias 0 -> 2
- net GPIO13: track 0.00 -> 57.4 mm, vias 0 -> 2
- net GPIO14: track 0.00 -> 53.6 mm, vias 0 -> 2
- net GPIO17: track 0.00 -> 39.2 mm, vias 0 -> 2
- net GPIO16: track 0.00 -> 38.1 mm, vias 0 -> 2
- net IO10P: track 0.00 -> 31.4 mm, vias 0 -> 2
- net AIO8N: track 0.00 -> 31.3 mm, vias 0 -> 1
- net IO5P: track 0.00 -> 31.2 mm, vias 0 -> 2
- net IO21P: track 0.00 -> 30.2 mm, vias 0 -> 1
- net POR_B: track 2.79 -> 32.9 mm
- net IO5N: track 0.00 -> 29.8 mm, vias 0 -> 2
- net IO4P: track 0.00 -> 29.0 mm, vias 0 -> 2
- net IO21N: track 0.00 -> 28.3 mm, vias 0 -> 1
- net IO11P: track 0.00 -> 28.0 mm, vias 0 -> 2
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- added copper zone on In2.Cu, net +3.3VA
- added copper zone on In1.Cu, net +5VD
- added copper zone on In4.Cu, net GND
- added copper zone on F.Cu, net VBUS0
- removed copper zone on In4.Cu, net +3V3
Other:
- board size 74.3 x 21 mm -> 84 x 20.9 mm
