File: DDR3 test/DDR3 test/FPGApwr.kicad_sch (KiCad schematic)
At the start: 20 parts, among them U3 XC7Z010-1CLG225I

Commit message: Resistor Footprints
- Fixed resistor footprints
- Re-added 3D models
- Routed 1.5V reg
Parts:
- R11, R12, R13: footprint Capacitor_SMD:C_0201_0603Metric -> Resistor_SMD:R_0201_0603Metric
- U3: footprint Sync_VT extras:225-LFBGA -> Sync_VT extras:BGA225C80P15X15_1300X1300X150N
Changed lines of the file:
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@@
 			)
 		)
-		(property "Footprint" "Capacitor_SMD:C_0201_0603Metric"
+		(property "Footprint" "Resistor_SMD:R_0201_0603Metric"
 			(at 111.76 36.322 90)
 			(effects
@@
 			)
 		)
-		(property "Footprint" "Sync_VT extras:225-LFBGA"
+		(property "Footprint" "Sync_VT extras:BGA225C80P15X15_1300X1300X150N"
 			(at 179.07 45.72 0)
 			(effects
@@
 			)
 		)
-		(property "Footprint" "Capacitor_SMD:C_0201_0603Metric"
+		(property "Footprint" "Resistor_SMD:R_0201_0603Metric"
 			(at 111.76 38.862 90)
 			(effects
@@
 			)
 		)
-		(property "Footprint" "Capacitor_SMD:C_0201_0603Metric"
+		(property "Footprint" "Resistor_SMD:R_0201_0603Metric"
 			(at 31.75 49.022 90)
 			(effects
@@
 			)
 		)
-		(property "Footprint" "Sync_VT extras:225-LFBGA"
+		(property "Footprint" "Sync_VT extras:BGA225C80P15X15_1300X1300X150N"
 			(at 77.47 48.26 0)
 			(effects
